Commit message: Fix mesh size unit, urdf

File: melfa_description/urdf/rv7fl.urdf.xacro (robot description, xacro)
@@ -29,125 +29,105 @@
   <link name="base_link">
     <visual>
-        <origin xyz="0 0 0" rpy="0 0 0"/>
-        <axis xyz="0 0 0"/>
-        <geometry>
-            <mesh filename="package://melfa_description/meshe/B.STL" scale="${MODEL_RATIO} ${MODEL_RATIO} ${MODEL_RATIO}"/>
-        </geometry>
-        <material name="grey"/>
+      <origin xyz="0 0 0" rpy="${pi/2} 0 0"/>
+      <axis xyz="0 0 0"/>
+      <geometry>
+        <mesh filename="package://melfa_description/mesh/RV-7F_BASE_01.stl"/>
+      </geometry>
+      <material name="grey"/>
     </visual>
   </link>
-  <!-- +++++++++++++++++++++++++++++++++++++++++++++++++++++++++++++++++joint1 -->
   <joint name="joint1" type="revolute">
     <parent link="base_link"/>
-    <child link="link_j1"/>
-    <origin xyz="${BASE_J1X} ${BASE_J1Y} ${BASE_J1Z}" rpy="0 0 0"/>
+    <child link="link1"/>
+    <origin xyz="0 0 0.4" rpy="0 0 0"/>
     <axis xyz="0 0 1"/>
     <dynamics damping="0.7"/>
     <limit upper="2.18" lower="-2.18" effort="10" velocity="1" />
   </joint>
-  <!-- ==================================================================link1 -->
-  <link name="link_j1">
+  <link name="link1">
     <visual>
-      <origin xyz="0 0 0" rpy="${RIGHT_ANGLE} 0 0"/>
+      <origin xyz="0 0 0" rpy="${pi/2} 0 0"/>
       <geometry>
-        <mesh filename="package://tra1_description/meshes/J1.STL" scale="${MODEL_RATIO} ${MODEL_RATIO} ${MODEL_RATIO}"/>
-      </geometry>
-      <material name="black"/>
-    </visual>
-  </link>
-  <!-- +++++++++++++++++++++++++++++++++++++++++++++++++++++++++++++++++joint2 -->
-  <joint name="joint2" type="revolute">
-    <parent link="link_j1"/>
-    <child link="link_j2"/>
-    <origin xyz="${J1X_J2X-BASE_J1X} ${J1Y_J2Y-BASE_J1Y} ${J1Z_J2Z-BASE_J1Z}" rpy="0 0 0"/>
-    <axis xyz="1 0 0"/>
-    <dynamics damping="0.7"/>
-    <limit upper="2.18" lower="-2.18" effort="10" velocity="1" />
-  </joint>
-  <!-- ==================================================================link2 -->
-  <link name="link_j2">
-    <visual>
-      <origin xyz="0 0 0" rpy="${RIGHT_ANGLE} 0 0"/>
-      <geometry>
-        <mesh filename="package://tra1_description/meshes/J2.STL" scale="${MODEL_RATIO} ${MODEL_RATIO} ${MODEL_RATIO}"/>
+        <mesh filename="package://melfa_description/mesh/RV-7F_SHOLDER_02.stl"/>
       </geometry>
       <material name="grey"/>
     </visual>
   </link>
-  <!-- +++++++++++++++++++++++++++++++++++++++++++++++++++++++++++++++++joint3 -->
-    <joint name="joint3" type="revolute">
-      <parent link="link_j2"/>
-      <child link="link_j3"/>
-      <origin xyz="${J2X_J3X-J1X_J2X} ${J2Y_J3Y-J1Y_J2Y} ${J2Z_J3Z-J1Z_J2Z}" rpy="0 0 0"/>
-      <axis xyz="1 0 0"/>
-      <dynamics damping="0.7"/>
-      <limit upper="2.18" lower="-2.18" effort="10" velocity="1" />
-    </joint>
-  <!-- ==================================================================link3 -->
-  <link name="link_j3">
+  <joint name="joint2" type="revolute">
+    <parent link="link1"/>
+    <child link="link2"/>
+    <origin xyz="0 0 0" rpy="0 0 0"/>
+    <axis xyz="0 1 0"/>
+    <dynamics damping="0.7"/>
+    <limit upper="2.18" lower="-2.18" effort="10" velocity="1" />
+  </joint>
+  <link name="link2">
     <visual>
-      <origin xyz="0 0 0" rpy="${RIGHT_ANGLE} 0 0"/>
+      <origin xyz="0 0 0" rpy="${pi/2} 0 0"/>
       <geometry>
-        <mesh filename="package://tra1_description/meshes/J3.STL" scale="${MODEL_RATIO} ${MODEL_RATIO} ${MODEL_RATIO}"/>
+        <mesh filename="package://melfa_description/mesh/RV_7FL_NO1ARM_03.stl"/>
       </geometry>
       <material name="grey"/>
     </visual>
   </link>
-  <!-- +++++++++++++++++++++++++++++++++++++++++++++++++++++++++++++++++joint4 -->
+  <joint name="joint3" type="revolute">
+    <parent link="link2"/>
+    <child link="link3"/>
+    <origin xyz="0 0 0.435" rpy="0 0 0"/>
+    <axis xyz="0 1 0"/>
+    <dynamics damping="0.7"/>
+    <limit upper="2.18" lower="-2.18" effort="10" velocity="1" />
+  </joint>
+  <link name="link3">
+    <visual>
+      <origin xyz="0 0 0" rpy="${pi/2} ${pi/2} 0"/>
+      <geometry>
+        <mesh filename="package://melfa_description/mesh/RV-7F_ELBOW_04.stl"/>
+      </geometry>
+      <material name="grey"/>
+    </visual>
+  </link>
   <joint name="joint4" type="revolute">
-    <parent link="link_j3"/>
-    <child link="link_j4"/>
-    <origin xyz="${J3X_J4X-J2X_J3X} ${J3Y_J4Y-J2Y_J3Y} ${J3Z_J4Z-J2Z_J3Z}" rpy="0 0 0"/>
+    <parent link="link3"/>
+    <child link="link4"/>
+    <origin xyz="0.05 0 0.47" rpy="0 0 0"/>
     <axis xyz="0 0 1"/>
     <dynamics damping="0.7"/>
     <limit upper="2.18" lower="-2.18" effort="10" velocity="1" />
   </joint>
-  <!-- ==================================================================link4 -->
-  <link name="link_j4">
+  <link name="link4">
     <visual>
-      <origin xyz="0 0 0" rpy="${RIGHT_ANGLE} 0 0"/>
+      <origin xyz="0 0 0" rpy="${-pi/2} ${pi/2} 0"/>
       <geometry>
-        <mesh filename="package://tra1_description/meshes/J4.STL" scale="${MODEL_RATIO} ${MODEL_RATIO} ${MODEL_RATIO}"/>
-      </geometry>
-      <material name="black"/>
-    </visual>
-  </link>
-  <!-- +++++++++++++++++++++++++++++++++++++++++++++++++++++++++++++++++joint5 -->
-  <joint name="joint5" type="revolute">
-    <parent link="link_j4"/>
-    <child link="link_j5"/>
-    <origin xyz="${J4X_J5X-J3X_J4X} ${J4Y_J5Y-J3Y_J4Y} ${J4Z_J5Z-J3Z_J4Z}" rpy="0 0 0"/>
-    <axis xyz="1 0 0"/>
-    <dynamics damping="0.7"/>
-    <limit upper="2.18" lower="-2.18" effort="10" velocity="1" />
-  </joint>
-  <!-- ==================================================================link5 -->
-  <link name="link_j5">
-    <visual>
-      <origin xyz="0 0 0" rpy="${RIGHT_ANGLE} 0 0"/>
-      <geometry>
-        <mesh filename="package://tra1_description/meshes/J5.STL" scale="${MODEL_RATIO} ${MODEL_RATIO} ${MODEL_RATIO}"/>
+        <mesh filename="package://melfa_description/mesh/RV_7FL_NO2ARM_05.stl"/>
       </geometry>
       <material name="grey"/>
     </visual>
   </link>
-  <!-- +++++++++++++++++++++++++++++++++++++++++++++++++++++++++++++++++joint6 -->
+  <joint name="joint5" type="revolute">
+    <parent link="link4"/>
+    <child link="link5"/>
+    <origin xyz="0 0 0" rpy="0 0 0"/>
+    <axis xyz="0 1 0"/>
+    <dynamics damping="0.7"/>
+    <limit upper="2.18" lower="-2.18" effort="10" velocity="1" />
+  </joint>
+  <link name="link5">
+    <visual>
+      <origin xyz="0 0 0" rpy="${-pi/2} ${pi/2} 0"/>
+      <geometry>
+        <mesh filename="package://melfa_description/mesh/RV-4F_WRIST_06.stl"/>
+      </geometry>
+      <material name="grey"/>
+    </visual>
+  </link>
   <joint name="joint6" type="revolute">
-    <parent link="link_j5"/>
-    <child link="link_j6"/>
-    <origin xyz="${J5X_J6X-J4X_J5X} ${J5Y_J6Y-J4Y_J5Y} ${J5Z_J6Z-J4Z_J5Z}" rpy="0 0 0"/>
+    <parent link="link5"/>
+    <child link="link6"/>
+    <origin xyz="0 0 0" rpy="0 0 0"/>
     <axis xyz="0 0 1"/>
     <dynamics damping="0.7"/>
     <limit upper="2.18" lower="-2.18" effort="10" velocity="1" />
   </joint>
-  <!-- ==================================================================link6 -->
-  <link name="link_j6">
-    <visual>
-      <origin xyz="0 0 0" rpy="${RIGHT_ANGLE} 0 0"/>
-      <geometry>
-        <mesh filename="package://tra1_description/meshes/J6.STL" scale="${MODEL_RATIO} ${MODEL_RATIO} ${MODEL_RATIO}"/>
-      </geometry>
-      <material name="black"/>
-    </visual>
-  </link>
+  <link name="link6"/>
 </robot>

Commit message: Modify joint limits to fit the spec sheet

File: melfa_description/urdf/rv7fl.urdf.xacro (robot description, xacro)
@@ -19,5 +19,5 @@
     <axis xyz="0 0 1"/>
     <dynamics damping="0.7"/>
-    <limit upper="2.18" lower="-2.18" effort="10" velocity="1" />
+    <limit upper="${240*pi/180}" lower="${-240*pi/180}" effort="10" velocity="${288*pi/180}" />
   </joint>
   <link name="link1">
@@ -36,5 +36,5 @@
     <axis xyz="0 1 0"/>
     <dynamics damping="0.7"/>
-    <limit upper="2.18" lower="-2.18" effort="10" velocity="1" />
+    <limit upper="${130*pi/180}" lower="${-110*pi/180}" effort="10" velocity="${321*pi/180}" />
   </joint>
   <link name="link2">
@@ -53,5 +53,5 @@
     <axis xyz="0 1 0"/>
     <dynamics damping="0.7"/>
-    <limit upper="2.18" lower="0.00" effort="10" velocity="1" />
+    <limit upper="${162*pi/180}" lower="0.00" effort="10" velocity="${360*pi/180}" />
   </joint>
   <link name="link3">
@@ -70,5 +70,5 @@
     <axis xyz="0 0 1"/>
     <dynamics damping="0.7"/>
-    <limit upper="2.18" lower="-2.18" effort="10" velocity="1" />
+    <limit upper="${200*pi/180}" lower="${-200*pi/180}" effort="10" velocity="${337*pi/180}" />
   </joint>
   <link name="link4">
@@ -87,5 +87,5 @@
     <axis xyz="0 1 0"/>
     <dynamics damping="0.7"/>
-    <limit upper="2.18" lower="-2.18" effort="10" velocity="1" />
+    <limit upper="${120*pi/180}" lower="${-120*pi/180}" effort="10" velocity="${450*pi/180}" />
   </joint>
   <link name="link5">
@@ -101,8 +101,8 @@
     <parent link="link5"/>
     <child link="link6"/>
-    <origin xyz="0 0 0" rpy="0 0 0"/>
+    <origin xyz="0 0 0.085" rpy="0 0 0"/>
     <axis xyz="0 0 1"/>
     <dynamics damping="0.7"/>
-    <limit upper="2.18" lower="-2.18" effort="10" velocity="1" />
+    <limit upper="${360*pi/180}" lower="${-360*pi/180}" effort="10" velocity="${720*pi/180}" />
   </joint>
   <link name="link6"/>

Commit message: Add dummy joint7 and joint8 for actual robot

File: melfa_description/urdf/rv7fl.urdf.xacro (robot description, xacro)
@@ -107,3 +107,19 @@
   </joint>
   <link name="link6"/>
+  <link name="dummy1"/>
+  <joint name="joint7" type="revolute">
+    <parent link="base_link"/>
+    <child link="dummy1"/>
+    <origin xyz="0 0 0" rpy="0 0 0"/>
+    <axis xyz="0 0 1"/>
+    <limit upper="${240*pi/180}" lower="${-240*pi/180}" effort="10" velocity="${288*pi/180}" />
+  </joint>
+  <link name="dummy2"/>
+  <joint name="joint8" type="revolute">
+    <parent link="base_link"/>
+    <child link="dummy2"/>
+    <origin xyz="0 0 0" rpy="0 0 0"/>
+    <axis xyz="0 0 1"/>
+    <limit upper="${240*pi/180}" lower="${-240*pi/180}" effort="10" velocity="${288*pi/180}" />
+  </joint>
 </robot>

Commit message: Remove mesh related files from melfa_description

File: melfa_description/urdf/rv7fl.urdf.xacro (robot description, xacro)
@@ -2,14 +2,5 @@
 <!-- Copyright (C) 2018, Tokyo Opensource Robotics Kyokai Association -->
 <robot name="rv7fl" xmlns:xacro="http://www.ros.org/wiki/xacro">
-  <xacro:include filename="$(find melfa_description)/urdf/materials.xacro" />
   <link name="base_link">
-    <visual>
-      <origin xyz="0 0 0" rpy="${pi/2} 0 ${pi}"/>
-      <axis xyz="0 0 0"/>
-      <geometry>
-        <mesh filename="package://melfa_description/mesh/RV-7F_BASE_01.stl"/>
-      </geometry>
-      <material name="white1"/>
-    </visual>
   </link>
   <joint name="joint1" type="revolute">
@@ -22,11 +13,4 @@
   </joint>
   <link name="link1">
-    <visual>
-      <origin xyz="0 0 0" rpy="${pi/2} 0 ${pi}"/>
-      <geometry>
-        <mesh filename="package://melfa_description/mesh/RV-7F_SHOLDER_02.stl"/>
-      </geometry>
-      <material name="white2"/>
-    </visual>
   </link>
   <joint name="joint2" type="revolute">
@@ -39,11 +23,4 @@
   </joint>
   <link name="link2">
-    <visual>
-      <origin xyz="0 0 0" rpy="${pi/2} 0 ${pi}"/>
-      <geometry>
-        <mesh filename="package://melfa_description/mesh/RV_7FL_NO1ARM_03.stl"/>
-      </geometry>
-      <material name="white3"/>
-    </visual>
   </link>
   <joint name="joint3" type="revolute">
@@ -56,11 +33,4 @@
   </joint>
   <link name="link3">
-    <visual>
-      <origin xyz="0 0 0" rpy="0 ${pi/2} ${pi/2}"/>
-      <geometry>
-        <mesh filename="package://melfa_description/mesh/RV-7F_ELBOW_04.stl"/>
-      </geometry>
-      <material name="white1"/>
-    </visual>
   </link>
   <joint name="joint4" type="revolute">
@@ -73,11 +43,4 @@
   </joint>
   <link name="link4">
-    <visual>
-      <origin xyz="0 0 0" rpy="0 ${pi/2} ${-pi/2}"/>
-      <geometry>
-        <mesh filename="package://melfa_description/mesh/RV_7FL_NO2ARM_05.stl"/>
-      </geometry>
-      <material name="white2"/>
-    </visual>
   </link>
   <joint name="joint5" type="revolute">
@@ -90,11 +53,4 @@
   </joint>
   <link name="link5">
-    <visual>
-      <origin xyz="0 0 0" rpy="0 ${pi/2} ${-pi/2}"/>
-      <geometry>
-        <mesh filename="package://melfa_description/mesh/RV-4F_WRIST_06.stl"/>
-      </geometry>
-      <material name="white3"/>
-    </visual>
   </link>
   <joint name="joint6" type="revolute">

Commit message: Add use_joint7 and use_joint8 parameters
- Remove dummy joints from rv7fl.urdf.xacro

File: melfa_description/urdf/rv7fl.urdf.xacro (robot description, xacro)
@@ -159,19 +159,3 @@
     </collision>
   </link>
-  <link name="dummy1"/>
-  <joint name="joint7" type="revolute">
-    <parent link="base_link"/>
-    <child link="dummy1"/>
-    <origin xyz="0 0 0" rpy="0 0 0"/>
-    <axis xyz="0 0 1"/>
-    <limit upper="${240*pi/180}" lower="${-240*pi/180}" effort="10" velocity="${288*pi/180}" />
-  </joint>
-  <link name="dummy2"/>
-  <joint name="joint8" type="revolute">
-    <parent link="base_link"/>
-    <child link="dummy2"/>
-    <origin xyz="0 0 0" rpy="0 0 0"/>
-    <axis xyz="0 0 1"/>
-    <limit upper="${240*pi/180}" lower="${-240*pi/180}" effort="10" velocity="${288*pi/180}" />
-  </joint>
 </robot>

Commit message: Organize rv7fl.urdf.xacro using xacro

File: melfa_description/urdf/rv7fl.urdf.xacro (robot description, xacro)
@@ -5,157 +5,8 @@
     <color rgba="1.0 1.0 1.0 1.0"/>
   </material>
-  <xacro:property name="folder" value="package://melfa_description/mesh/rv7fl"/>
-  <link name="base_link">
-    <visual>
-      <origin rpy="0 0 0" xyz="0 0 0"/>
-      <geometry>
-	<mesh filename="package://melfa_description/mesh/rv7fl/L0.stl" scale="1.4 1.4 1.1"/>
-      </geometry>
-      <material name="white"/>
-    </visual>
-    <collision>
-      <origin rpy="0 0 0" xyz="0 0 0"/>
-      <geometry>
-	<mesh filename="package://melfa_description/mesh/rv7fl/L0.stl" scale="1.4 1.4 1.1"/>
-      </geometry>
-    </collision>
-  </link>
-  <joint name="joint1" type="revolute">
-    <parent link="base_link"/>
-    <child link="link1"/>
-    <origin xyz="0 0 0.4" rpy="0 0 0"/>
-    <axis xyz="0 0 1"/>
-    <dynamics damping="0.7"/>
-    <limit upper="${240*pi/180}" lower="${-240*pi/180}" effort="10" velocity="${288*pi/180}" />
-  </joint>
-  <link name="link1">
-    <visual>
-      <origin rpy="0 0 0" xyz="0 0 0"/>
-      <geometry>
-	<mesh filename="package://melfa_description/mesh/rv7fl/L1.stl" scale="1.3 1.3 1.3"/>
-      </geometry>
-      <material name="white"/>
-    </visual>
-    <collision>
-      <origin rpy="0 0 0" xyz="0 0 0"/>
-      <geometry>
-	<mesh filename="package://melfa_description/mesh/rv7fl/L1.stl" scale="1.3 1.3 1.3"/>
-      </geometry>
-    </collision>
-  </link>
-  <joint name="joint2" type="revolute">
-    <parent link="link1"/>
-    <child link="link2"/>
+  <xacro:include filename="$(find melfa_description)/urdf/rv7fl.xacro"/>
+  <link name="base_link"/>
+  <xacro:rv7fl parent="base_link">
     <origin xyz="0 0 0" rpy="0 0 0"/>
-    <axis xyz="0 1 0"/>
-    <dynamics damping="0.7"/>
-    <limit upper="${130*pi/180}" lower="${-110*pi/180}" effort="10" velocity="${321*pi/180}" />
-  </joint>
-  <link name="link2">
-    <visual>
-      <origin rpy="0 0 0" xyz="0 0 0"/>
-      <geometry>
-	<mesh filename="package://melfa_description/mesh/rv7fl/L2.stl" scale="1.45 1.45 1.45"/>
-      </geometry>
-      <material name="white"/>
-    </visual>
-    <collision>
-      <origin rpy="0 0 0" xyz="0 0 0"/>
-      <geometry>
-	<mesh filename="package://melfa_description/mesh/rv7fl/L2.stl" scale="1.45 1.45 1.45"/>
-      </geometry>
-    </collision>
-  </link>
-  <joint name="joint3" type="revolute">
-    <parent link="link2"/>
-    <child link="link3"/>
-    <origin xyz="0 0 0.435" rpy="0 0 0"/>
-    <axis xyz="0 1 0"/>
-    <dynamics damping="0.7"/>
-    <limit upper="${162*pi/180}" lower="0.00" effort="10" velocity="${360*pi/180}" />
-  </joint>
-  <link name="link3">
-    <visual>
-      <origin rpy="0 0 0" xyz="0 0 0"/>
-      <geometry>
-	<mesh filename="package://melfa_description/mesh/rv7fl/L3.stl" scale="1.3 1.3 1.3"/>
-      </geometry>
-      <material name="white"/>
-    </visual>
-    <collision>
-      <origin rpy="0 0 0" xyz="0 0 0"/>
-      <geometry>
-	<mesh filename="package://melfa_description/mesh/rv7fl/L3.stl" scale="1.3 1.3 1.3"/>
-      </geometry>
-    </collision>
-  </link>
-  <joint name="joint4" type="revolute">
-    <parent link="link3"/>
-    <child link="link4"/>
-    <origin xyz="-0.05 0 0.47" rpy="0 0 0"/>
-    <axis xyz="0 0 1"/>
-    <dynamics damping="0.7"/>
-    <limit upper="${200*pi/180}" lower="${-200*pi/180}" effort="10" velocity="${337*pi/180}" />
-  </joint>
-  <link name="link4">
-    <visual>
-      <origin rpy="0 0 0" xyz="0 0 0"/>
-      <geometry>
-	<mesh filename="package://melfa_description/mesh/rv7fl/L4.stl" scale="1.4 1.4 1.4"/>
-      </geometry>
-      <material name="white"/>
-    </visual>
-    <collision>
-      <origin rpy="0 0 0" xyz="0 0 0"/>
-      <geometry>
-	<mesh filename="package://melfa_description/mesh/rv7fl/L4.stl" scale="1.4 1.4 1.4"/>
-      </geometry>
-    </collision>
-  </link>
-  <joint name="joint5" type="revolute">
-    <parent link="link4"/>
-    <child link="link5"/>
-    <origin xyz="0 0 0" rpy="0 0 0"/>
-    <axis xyz="0 1 0"/>
-    <dynamics damping="0.7"/>
-    <limit upper="${120*pi/180}" lower="${-120*pi/180}" effort="10" velocity="${450*pi/180}" />
-  </joint>
-  <link name="link5">
-    <visual>
-      <origin rpy="0 0 0" xyz="0 0 0"/>
-      <geometry>
-	<mesh filename="package://melfa_description/mesh/rv7fl/L5.stl" scale="1.4 1.4 1.4"/>
-      </geometry>
-      <material name="white"/>
-    </visual>
-    <collision>
-      <origin rpy="0 0 0" xyz="0 0 0"/>
-      <geometry>
-	<mesh filename="package://melfa_description/mesh/rv7fl/L5.stl" scale="1.4 1.4 1.4"/>
-      </geometry>
-    </collision>
-  </link>
-  <joint name="joint6" type="revolute">
-    <parent link="link5"/>
-    <child link="link6"/>
-    <origin xyz="0 0 0.085" rpy="0 0 0"/>
-    <axis xyz="0 0 1"/>
-    <dynamics damping="0.7"/>
-    <limit upper="${360*pi/180}" lower="${-360*pi/180}" effort="10" velocity="${720*pi/180}" />
-  </joint>
-  <link name="link6">
-    <visual>
-      <origin rpy="0 0 0" xyz="0 0 0"/>
-      <geometry>
-	<mesh filename="package://melfa_description/mesh/rv7fl/L6.stl"/>
-      </geometry>
-      <material name="white"/>
-    </visual>
-    <collision>
-      <origin rpy="0 0 0" xyz="0 0 0"/>
-      <geometry>
-	<mesh filename="package://melfa_description/mesh/rv7fl/L6.stl"/>
-      </geometry>
-    </collision>
-  </link>
+  </xacro:rv7fl>
 </robot>
