Commit message: Modify URDF to adopt the package structure
- Add robot argument to specify target robot

File: melfa_description/urdf/rv4fl.urdf.xacro (robot description, xacro)
@@ -1,19 +1,20 @@
 <?xml version="1.0"?>
-<robot xmlns:xacro="http://www.ros.org/wiki/xacro" name="test_robot">
-	<material name="black">
-		<color rgba="0.0 0.0 0.0 1.0"/>
-	</material>
-	<material name="white">
-		<color rgba="1.0 1.0 1.0 1.0"/>
-	</material>
-	<material name="yoods">
-		<color rgba="1.0 1.0 0.7 0.9"/>
-	</material>
-	<!--~~~~~~~~~~~~~~~~~~~~~~~~~~~~~~~~-->
-	<!-- macro -->
-	<!--~~~~~~~~~~~~~~~~~~~~~~~~~~~~~~~~-->
-	<xacro:property name="pi" value="3.1415926535897931" />
+<!-- Copyright (C) 2018, YOODS, Inc. -->
+<robot name="rv4fl" xmlns:xacro="http://www.ros.org/wiki/xacro">
+  <material name="black">
+    <color rgba="0.0 0.0 0.0 1.0"/>
+  </material>
+  <material name="white">
+    <color rgba="1.0 1.0 1.0 1.0"/>
+  </material>
+  <material name="yoods">
+    <color rgba="1.0 1.0 0.7 0.9"/>
+  </material>
+  <!--~~~~~~~~~~~~~~~~~~~~~~~~~~~~~~~~-->
+  <!-- macro -->
+  <!--~~~~~~~~~~~~~~~~~~~~~~~~~~~~~~~~-->
+  <xacro:property name="pi" value="3.1415926535897931" />
   <!-- STL file -->
-	<xacro:property name="folder" value="package://robot_model/rv4fl"/>
+  <xacro:property name="folder" value="package://melfa_description/mesh/rv4fl"/>
   <xacro:property name="link0_stl" value="${folder}/L0.stl" />
   <xacro:property name="link1_stl" value="${folder}/L1.stl" />
@@ -23,62 +24,62 @@
   <xacro:property name="link5_stl" value="${folder}/L5.stl" />
   <xacro:property name="link6_stl" value="${folder}/L6.stl" />
-  <xacro:property name="handeye_stl" value="package://robot_model/equipment/handEye.stl" />
+  <xacro:property name="handeye_stl" value="package://melfa_description/mesh/equipment/handEye.stl" />
   <!-- STL model yawing -->
   <xacro:property name="yaw" value="${pi}"/>
   <!-- link definition -->
   <xacro:macro name="link_visual" params="fn col origin_xyz">
-		<visual>
-			<geometry>
-				<mesh filename="${fn}"/>
-			</geometry>
-			<material name="${col}"/>
+    <visual>
+      <geometry>
+	<mesh filename="${fn}"/>
+      </geometry>
+      <material name="${col}"/>
       <origin rpy="0 0 ${yaw}" xyz="${origin_xyz}"/>
-		</visual>
-		<collision>
-			<geometry>
-				<mesh filename="${fn}"/>
-			</geometry>
+    </visual>
+    <collision>
+      <geometry>
+	<mesh filename="${fn}"/>
+      </geometry>
       <origin rpy="0 0 ${yaw}" xyz="${origin_xyz}"/>
-		</collision>
-	</xacro:macro>
-	<xacro:macro name="link_state" params="mass origin_xyz ixx ixy ixz iyy iyz izz">
-		<inertial>
-			<mass value="${mass}"/>
-			<origin rpy="0 0 0" xyz="${origin_xyz}"/>
-			<inertia ixx="${ixx}" ixy="${ixy}" ixz="${ixz}"
-                            iyy="${iyy}" iyz="${iyz}"
-                                         izz="${izz}"/>
-		</inertial>
-	</xacro:macro>
+    </collision>
+  </xacro:macro>
+  <xacro:macro name="link_state" params="mass origin_xyz ixx ixy ixz iyy iyz izz">
+    <inertial>
+      <mass value="${mass}"/>
+      <origin rpy="0 0 0" xyz="${origin_xyz}"/>
+      <inertia ixx="${ixx}" ixy="${ixy}" ixz="${ixz}"
+               iyy="${iyy}" iyz="${iyz}"
+               izz="${izz}"/>
+    </inertial>
+  </xacro:macro>
   <!-- joint definition -->
-	<xacro:macro name="joint_state" params="parent child origin_xyz axis effort lower upper vel">
-		<parent link="${parent}"/>
-		<child link="${child}"/>
-		<origin rpy="0 0 0" xyz="${origin_xyz}"/>
-		<axis xyz="${axis}"/>
-		<limit effort="${effort}" lower="${lower}" upper="${upper}" velocity="${vel}"/>
-	</xacro:macro>
-	<!--~~~~~~~~~~~~~~~~~~~~~~~~~~~~~~~-->
-	<!-- world -->
-	<!--~~~~~~~~~~~~~~~~~~~~~~~~~~~~~~~-->
-	<link name="world"/>
-	<!-- fixed joint -->
-	<joint name="world_joint" type="fixed">
-		<parent link="world"/>
-		<child link="base_link"/>
-	</joint>
-	<!--~~~~~~~~~~~~~~~~~~~~~~~~~~~~~~~-->
-	<!-- base_link -->
-	<!--~~~~~~~~~~~~~~~~~~~~~~~~~~~~~~~-->
-	<link name="base_link">
-		<origin rpy="0 0 ${pi}"/>
+  <xacro:macro name="joint_state" params="parent child origin_xyz axis effort lower upper vel">
+    <parent link="${parent}"/>
+    <child link="${child}"/>
+    <origin rpy="0 0 0" xyz="${origin_xyz}"/>
+    <axis xyz="${axis}"/>
+    <limit effort="${effort}" lower="${lower}" upper="${upper}" velocity="${vel}"/>
+  </xacro:macro>
+  <!--~~~~~~~~~~~~~~~~~~~~~~~~~~~~~~~-->
+  <!-- world -->
+  <!--~~~~~~~~~~~~~~~~~~~~~~~~~~~~~~~-->
+  <link name="world"/>
+  <!-- fixed joint -->
+  <joint name="world_joint" type="fixed">
+    <parent link="world"/>
+    <child link="base_link"/>
+  </joint>
+  <!--~~~~~~~~~~~~~~~~~~~~~~~~~~~~~~~-->
+  <!-- base_link -->
+  <!--~~~~~~~~~~~~~~~~~~~~~~~~~~~~~~~-->
+  <link name="base_link">
+    <origin rpy="0 0 ${pi}"/>
     <xacro:link_visual fn="${link0_stl}"
                        col="white"
                        origin_xyz="0 0 0"/>
-	</link>
-	<!--~~~~~~~~~~~~~~~~~~~~~~~~~~~~~~~-->
-	<!-- joint 1 -->
-	<!--~~~~~~~~~~~~~~~~~~~~~~~~~~~~~~~-->
-	<joint name="joint1" type="revolute">
+  </link>
+  <!--~~~~~~~~~~~~~~~~~~~~~~~~~~~~~~~-->
+  <!-- joint 1 -->
+  <!--~~~~~~~~~~~~~~~~~~~~~~~~~~~~~~~-->
+  <joint name="joint1" type="revolute">
     <xacro:joint_state parent="base_link"
                        child="link1"
@@ -89,10 +90,10 @@
                        upper="${ 240.*pi/180.}"
                        vel="7.330"/>
-		<dynamics damping="0.7"/>
-	</joint>
-	<!--~~~~~~~~~~~~~~~~~~~~~~~~~~~~~~~-->
-	<!-- link1 -->
-	<!--~~~~~~~~~~~~~~~~~~~~~~~~~~~~~~~-->
-	<link name="link1">
+    <dynamics damping="0.7"/>
+  </joint>
+  <!--~~~~~~~~~~~~~~~~~~~~~~~~~~~~~~~-->
+  <!-- link1 -->
+  <!--~~~~~~~~~~~~~~~~~~~~~~~~~~~~~~~-->
+  <link name="link1">
     <xacro:link_visual fn="${link1_stl}"
                        col="white"
@@ -100,9 +101,9 @@
                                    0
                                    -0.193"/>
-	</link>
-	<!--~~~~~~~~~~~~~~~~~~~~~~~~~~~~~~~-->
-	<!-- joint 2 -->
-	<!--~~~~~~~~~~~~~~~~~~~~~~~~~~~~~~~-->
-	<joint name="joint2" type="revolute">
+  </link>
+  <!--~~~~~~~~~~~~~~~~~~~~~~~~~~~~~~~-->
+  <!-- joint 2 -->
+  <!--~~~~~~~~~~~~~~~~~~~~~~~~~~~~~~~-->
+  <joint name="joint2" type="revolute">
     <xacro:joint_state parent="link1"
                        child="link2"
@@ -113,10 +114,10 @@
                        upper="${ 120.*pi/180.}"
                        vel="5.864"/>
-		<dynamics damping="0.7"/>
-	</joint>
-	<!--~~~~~~~~~~~~~~~~~~~~~~~~~~~~~~~-->
-	<!-- link2 -->
-	<!--~~~~~~~~~~~~~~~~~~~~~~~~~~~~~~~-->
-	<link name="link2">
+    <dynamics damping="0.7"/>
+  </joint>
+  <!--~~~~~~~~~~~~~~~~~~~~~~~~~~~~~~~-->
+  <!-- link2 -->
+  <!--~~~~~~~~~~~~~~~~~~~~~~~~~~~~~~~-->
+  <link name="link2">
     <xacro:link_visual fn="${link2_stl}"
                        col="white"
@@ -124,9 +125,9 @@
                                    -0.091
                                    ${-0.193-0.157}"/>
-	</link>
-	<!--~~~~~~~~~~~~~~~~~~~~~~~~~~~~~~~-->
-	<!-- joint 3 -->
-	<!--~~~~~~~~~~~~~~~~~~~~~~~~~~~~~~~-->
-	<joint name="joint3" type="revolute">
+  </link>
+  <!--~~~~~~~~~~~~~~~~~~~~~~~~~~~~~~~-->
+  <!-- joint 3 -->
+  <!--~~~~~~~~~~~~~~~~~~~~~~~~~~~~~~~-->
+  <joint name="joint3" type="revolute">
     <xacro:joint_state parent="link2"
                        child="link3"
@@ -137,10 +138,10 @@
                        upper="${164.*pi/180.}"
                        vel="4.363"/>
-		<dynamics damping="0.7"/>
-	</joint>
-	<!--~~~~~~~~~~~~~~~~~~~~~~~~~~~~~~~-->
-	<!-- link3 -->
-	<!--~~~~~~~~~~~~~~~~~~~~~~~~~~~~~~~-->
-	<link name="link3">
+    <dynamics damping="0.7"/>
+  </joint>
+  <!--~~~~~~~~~~~~~~~~~~~~~~~~~~~~~~~-->
+  <!-- link3 -->
+  <!--~~~~~~~~~~~~~~~~~~~~~~~~~~~~~~~-->
+  <link name="link3">
     <xacro:link_visual fn="${link3_stl}"
                        col="white"
@@ -148,9 +149,9 @@
                                    ${-0.091+0.047}
                                    ${-0.193-0.157-0.310}"/>
-	</link>
-	<!--~~~~~~~~~~~~~~~~~~~~~~~~~~~~~~~-->
-	<!-- joint 4 -->
-	<!--~~~~~~~~~~~~~~~~~~~~~~~~~~~~~~~-->
-	<joint name="joint4" type="revolute">
+  </link>
+  <!--~~~~~~~~~~~~~~~~~~~~~~~~~~~~~~~-->
+  <!-- joint 4 -->
+  <!--~~~~~~~~~~~~~~~~~~~~~~~~~~~~~~~-->
+  <joint name="joint4" type="revolute">
     <xacro:joint_state parent="link3"
                        child="link4"
@@ -161,10 +162,10 @@
                        upper="${ 200.*pi/180.}"
                        vel="9.425"/>
-		<dynamics damping="0.7"/>
-	</joint>
-	<!--~~~~~~~~~~~~~~~~~~~~~~~~~~~~~~~-->
-	<!-- link4 -->
-	<!--~~~~~~~~~~~~~~~~~~~~~~~~~~~~~~~-->
-	<link name="link4">
+    <dynamics damping="0.7"/>
+  </joint>
+  <!--~~~~~~~~~~~~~~~~~~~~~~~~~~~~~~~-->
+  <!-- link4 -->
+  <!--~~~~~~~~~~~~~~~~~~~~~~~~~~~~~~~-->
+  <link name="link4">
     <xacro:link_visual fn="${link4_stl}"
                        col="white"
@@ -172,9 +173,9 @@
                                    ${-0.091+0.047+0.044}
                                    ${-0.193-0.157-0.310-0.065}"/>
-	</link>
-	<!--~~~~~~~~~~~~~~~~~~~~~~~~~~~~~~~-->
-	<!-- joint 5 -->
-	<!--~~~~~~~~~~~~~~~~~~~~~~~~~~~~~~~-->
-	<joint name="joint5" type="revolute">
+  </link>
+  <!--~~~~~~~~~~~~~~~~~~~~~~~~~~~~~~~-->
+  <!-- joint 5 -->
+  <!--~~~~~~~~~~~~~~~~~~~~~~~~~~~~~~~-->
+  <joint name="joint5" type="revolute">
     <xacro:joint_state parent="link4"
                        child="link5"
@@ -185,10 +186,10 @@
                        upper="${ 120.*pi/180.}"
                        vel="10.875"/>
-		<dynamics damping="0.7"/>
-	</joint>
-	<!--~~~~~~~~~~~~~~~~~~~~~~~~~~~~~~~-->
-	<!-- link5 -->
-	<!--~~~~~~~~~~~~~~~~~~~~~~~~~~~~~~~-->
-	<link name="link5">
+    <dynamics damping="0.7"/>
+  </joint>
+  <!--~~~~~~~~~~~~~~~~~~~~~~~~~~~~~~~-->
+  <!-- link5 -->
+  <!--~~~~~~~~~~~~~~~~~~~~~~~~~~~~~~~-->
+  <link name="link5">
     <xacro:link_visual fn="${link5_stl}"
                        col="white"
@@ -196,9 +197,9 @@
                                    ${-0.091+0.047+0.044+0.021}
                                    ${-0.193-0.157-0.310-0.065-0.27}"/>
-	</link>
-	<!--~~~~~~~~~~~~~~~~~~~~~~~~~~~~~~~-->
-	<!-- joint 6 -->
-	<!--~~~~~~~~~~~~~~~~~~~~~~~~~~~~~~~-->
-	<joint name="joint6" type="revolute">
+  </link>
+  <!--~~~~~~~~~~~~~~~~~~~~~~~~~~~~~~~-->
+  <!-- joint 6 -->
+  <!--~~~~~~~~~~~~~~~~~~~~~~~~~~~~~~~-->
+  <joint name="joint6" type="revolute">
     <xacro:joint_state parent="link5"
                        child="link6"
@@ -209,10 +210,10 @@
                        upper="${ 200.*pi/180.}"
                        vel="12.566"/>
-		<dynamics damping="0.7"/>
-	</joint>
-	<!--~~~~~~~~~~~~~~~~~~~~~~~~~~~~~~~-->
-	<!-- link6 -->
-	<!--~~~~~~~~~~~~~~~~~~~~~~~~~~~~~~~-->
-	<link name="link6">
+    <dynamics damping="0.7"/>
+  </joint>
+  <!--~~~~~~~~~~~~~~~~~~~~~~~~~~~~~~~-->
+  <!-- link6 -->
+  <!--~~~~~~~~~~~~~~~~~~~~~~~~~~~~~~~-->
+  <link name="link6">
     <xacro:link_visual fn="${link6_stl}"
                        col="white"
@@ -220,9 +221,9 @@
                                    ${-0.091+0.047+0.044+0.021-0.021}
                                    ${-0.193-0.157-0.310-0.065-0.27-0.125}"/>
-	</link>
-	<!--~~~~~~~~~~~~~~~~~~~~~~~~~~~~~~~-->
-	<!-- joint 7 -->
-	<!--~~~~~~~~~~~~~~~~~~~~~~~~~~~~~~~-->
-	<joint name="joint7" type="fixed">
+  </link>
+  <!--~~~~~~~~~~~~~~~~~~~~~~~~~~~~~~~-->
+  <!-- joint 7 -->
+  <!--~~~~~~~~~~~~~~~~~~~~~~~~~~~~~~~-->
+  <joint name="joint7" type="fixed">
     <xacro:joint_state parent="link6"
                        child="handeye"
@@ -233,12 +234,12 @@
                        upper="0.0"
                        vel="0.0"/>
-	</joint>
-	<!--~~~~~~~~~~~~~~~~~~~~~~~~~~~~~~~-->
-	<!-- hand-eye -->
-	<!--~~~~~~~~~~~~~~~~~~~~~~~~~~~~~~~-->
-	<link name="handeye">
+  </joint>
+  <!--~~~~~~~~~~~~~~~~~~~~~~~~~~~~~~~-->
+  <!-- hand-eye -->
+  <!--~~~~~~~~~~~~~~~~~~~~~~~~~~~~~~~-->
+  <link name="handeye">
     <xacro:link_visual fn="${handeye_stl}"
                        col="yoods"
                        origin_xyz="0 0 0"/>
-	</link>
+  </link>
 </robot>

File: melfa_description/urdf/rv7fl.urdf.xacro (robot description, xacro)
@@ -2,5 +2,22 @@
 <!-- Copyright (C) 2018, Tokyo Opensource Robotics Kyokai Association -->
 <robot name="rv7fl" xmlns:xacro="http://www.ros.org/wiki/xacro">
+  <material name="white">
+    <color rgba="1.0 1.0 1.0 1.0"/>
+  </material>
+  <xacro:property name="folder" value="package://melfa_description/mesh/rv7fl"/>
   <link name="base_link">
+    <visual>
+      <origin rpy="0 0 0" xyz="0 0 0"/>
+      <geometry>
+	<mesh filename="package://melfa_description/mesh/rv7fl/L0.stl" scale="1.4 1.4 1.1"/>
+      </geometry>
+      <material name="white"/>
+    </visual>
+    <collision>
+      <origin rpy="0 0 0" xyz="0 0 0"/>
+      <geometry>
+	<mesh filename="package://melfa_description/mesh/rv7fl/L0.stl" scale="1.4 1.4 1.1"/>
+      </geometry>
+    </collision>
   </link>
   <joint name="joint1" type="revolute">
@@ -13,4 +30,17 @@
   </joint>
   <link name="link1">
+    <visual>
+      <origin rpy="0 0 0" xyz="0 0 0"/>
+      <geometry>
+	<mesh filename="package://melfa_description/mesh/rv7fl/L1.stl" scale="1.3 1.3 1.3"/>
+      </geometry>
+      <material name="white"/>
+    </visual>
+    <collision>
+      <origin rpy="0 0 0" xyz="0 0 0"/>
+      <geometry>
+	<mesh filename="package://melfa_description/mesh/rv7fl/L1.stl" scale="1.3 1.3 1.3"/>
+      </geometry>
+    </collision>
   </link>
   <joint name="joint2" type="revolute">
@@ -23,4 +53,17 @@
   </joint>
   <link name="link2">
+    <visual>
+      <origin rpy="0 0 0" xyz="0 0 0"/>
+      <geometry>
+	<mesh filename="package://melfa_description/mesh/rv7fl/L2.stl" scale="1.45 1.45 1.45"/>
+      </geometry>
+      <material name="white"/>
+    </visual>
+    <collision>
+      <origin rpy="0 0 0" xyz="0 0 0"/>
+      <geometry>
+	<mesh filename="package://melfa_description/mesh/rv7fl/L2.stl" scale="1.45 1.45 1.45"/>
+      </geometry>
+    </collision>
   </link>
   <joint name="joint3" type="revolute">
@@ -33,4 +76,17 @@
   </joint>
   <link name="link3">
+    <visual>
+      <origin rpy="0 0 0" xyz="0 0 0"/>
+      <geometry>
+	<mesh filename="package://melfa_description/mesh/rv7fl/L3.stl" scale="1.3 1.3 1.3"/>
+      </geometry>
+      <material name="white"/>
+    </visual>
+    <collision>
+      <origin rpy="0 0 0" xyz="0 0 0"/>
+      <geometry>
+	<mesh filename="package://melfa_description/mesh/rv7fl/L3.stl" scale="1.3 1.3 1.3"/>
+      </geometry>
+    </collision>
   </link>
   <joint name="joint4" type="revolute">
@@ -43,4 +99,17 @@
   </joint>
   <link name="link4">
+    <visual>
+      <origin rpy="0 0 0" xyz="0 0 0"/>
+      <geometry>
+	<mesh filename="package://melfa_description/mesh/rv7fl/L4.stl" scale="1.4 1.4 1.4"/>
+      </geometry>
+      <material name="white"/>
+    </visual>
+    <collision>
+      <origin rpy="0 0 0" xyz="0 0 0"/>
+      <geometry>
+	<mesh filename="package://melfa_description/mesh/rv7fl/L4.stl" scale="1.4 1.4 1.4"/>
+      </geometry>
+    </collision>
   </link>
   <joint name="joint5" type="revolute">
@@ -53,4 +122,17 @@
   </joint>
   <link name="link5">
+    <visual>
+      <origin rpy="0 0 0" xyz="0 0 0"/>
+      <geometry>
+	<mesh filename="package://melfa_description/mesh/rv7fl/L5.stl" scale="1.4 1.4 1.4"/>
+      </geometry>
+      <material name="white"/>
+    </visual>
+    <collision>
+      <origin rpy="0 0 0" xyz="0 0 0"/>
+      <geometry>
+	<mesh filename="package://melfa_description/mesh/rv7fl/L5.stl" scale="1.4 1.4 1.4"/>
+      </geometry>
+    </collision>
   </link>
   <joint name="joint6" type="revolute">
@@ -62,5 +144,19 @@
     <limit upper="${360*pi/180}" lower="${-360*pi/180}" effort="10" velocity="${720*pi/180}" />
   </joint>
-  <link name="link6"/>
+  <link name="link6">
+    <visual>
+      <origin rpy="0 0 0" xyz="0 0 0"/>
+      <geometry>
+	<mesh filename="package://melfa_description/mesh/rv7fl/L6.stl"/>
+      </geometry>
+      <material name="white"/>
+    </visual>
+    <collision>
+      <origin rpy="0 0 0" xyz="0 0 0"/>
+      <geometry>
+	<mesh filename="package://melfa_description/mesh/rv7fl/L6.stl"/>
+      </geometry>
+    </collision>
+  </link>
   <link name="dummy1"/>
   <joint name="joint7" type="revolute">
